Commit message: fixing eef

File: urdf/so101.urdf (robot description, URDF)
Before this commit: robot so101_leader_new_calib, 8 links, 7 joints
Links:
- link gripper_link: geometry collision mesh filename=package://so101_leader_description/meshes/handle_so101.stl scale=0.001 0.001 0.001; collision mesh filename=package://so101_leader_description/meshes/sts3215_03a_v1.stl
Joints:
- joint gripper: limit lower=-0.174533 upper=1.74533 effort=10 velocity=10 -> lower=-1.174533 upper=1.74533 effort=10 velocity=10
